File: src/HardwareDesign/1.0.0/BladeCore-M54C.kicad_pcb (KiCad board)
At the start: 6 copper layers, 29 x 80.6 mm, 132 parts, among them IC1 RP2354B, IC2 AT24C256C-XHL-T, IC29 TCAN1044AVDRBRQ1, IC3 W25Q128JVPIQ, IC4 MCP6001RT, IC5 LM4040B30FTA, IC6 MCP2515T-I/ML, IC7 TPS74801DRCT, IC8 SN74LVC1G97QDCKRQ1, IC9 FSUSB42MUX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

Commit message: Update M54C
Parts:
- added R39: 1R 1%, Resistor_SMD:R_0402_1005Metric, B.Cu at (220.4, 147.9)
- added R40: 1R 1%, Resistor_SMD:R_0402_1005Metric, B.Cu at (216.1, 147.9)
Routing:
- net /Project Architecture/CAN Interface/IC_CAN_N: track 4.18 -> 6.92 mm
- net /Project Architecture/CAN Interface/IC_CAN_P: track 4.18 -> 6.87 mm
- net /Project Architecture/CAN Interface/CAN_TERM_P: track 4.36 -> 4.39 mm, vias 0 -> 1
- net /Project Architecture/CAN Interface/CAN_TERM_N: vias 0 -> 1

Commit message: Finalize design
Parts:
- removed C54: 1uF 50V, Capacitor_SMD:C_0402_1005Metric
- added C36: 4.7uF 25V, Capacitor_SMD:C_0402_1005Metric, F.Cu at (214.2, 98.9)
- added D10: Green, LED_SMD:LED_0402_1005Metric, F.Cu at (234.1, 93.4)
- added R41: 1K 1%, Resistor_SMD:R_0402_1005Metric, F.Cu at (234.1, 92.0)
Connections:
- net /Project Architecture/USB Interface and Power/USB_IND renamed /Project Architecture/USB Interface and Power/5V_IND
- D2 pad 2: VBUS -> +5V
- IC7 pad 4: /Project Architecture/USB Interface and Power/BIAS -> +5V
Routing:
- net +5V: track 73.3 -> 87.9 mm, vias 11 -> 13
- net /Project Architecture/USB Interface and Power/USB_IND: track 0.00 -> 1.45 mm
- net /Project Architecture/USB Interface and Power/BIAS: track 1.38 -> 0.00 mm
- net VBUS_ONBOARD: track 44.3 -> 45.4 mm
- net VBUS: track 94.5 -> 93.8 mm
Other:
- board text added: "+5V"
- board text added: "USB"
- board text removed: "VBUS"

Commit message: add simple software
Connections:
- net /Project Architecture/Microcontroller/USB_IND renamed /Project Architecture/Microcontroller/HB_IND
Changed lines of the file:
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@@
 	(net 25 "QSPI_SD1")
 	(net 26 "/Project Architecture/USB Interface and Power/USB_IND")
-	(net 27 "/Project Architecture/Microcontroller/USB_IND")
+	(net 27 "/Project Architecture/Microcontroller/HB_IND")
 	(net 28 "QSPI_SS")
 	(net 29 "/Project Architecture/Microcontroller Peripherals/RP_D-")
@@
 			)
 		)
-		(property "LCSC_PART" "C26178"
-			(at 0 0 0)
-			(unlocked yes)
-			(layer "F.Fab")
-			(hide yes)
-			(effects
-				(font
-					(size 1 1)
-					(thickness 0.15)
-				)
-			)
-		)
 		(property ki_fp_filters "D*SMA*")
 		(sheetname "/Project Architecture/USB Interface and Power/")
@@
 		(sheetname "/Project Architecture/")
 		(sheetfile "Project Architecture.kicad_sch")
-		(attr smd)
+		(attr smd exclude_from_bom dnp)
 		(fp_line
 			(start -0.727064 0.91)
@@
 			(layers "F.Cu" "F.Mask" "F.Paste")
 			(roundrect_rratio 0.25)
-			(net 27 "/Project Architecture/Microcontroller/USB_IND")
+			(net 27 "/Project Architecture/Microcontroller/HB_IND")
 			(pintype "passive")
 		)
@@
 			(layers "F.Cu" "F.Mask" "F.Paste")
 			(roundrect_rratio 0.25)
-			(net 27 "/Project Architecture/Microcontroller/USB_IND")
+			(net 27 "/Project Architecture/Microcontroller/HB_IND")
 			(pintype "passive")
 		)
@@
 			)
 		)
-		(property "LCSC_PART" "C26178"
-			(at 0 0 0)
-			(unlocked yes)
-			(layer "B.Fab")
-			(hide yes)
-			(effects
-				(font
-					(size 1 1)
-					(thickness 0.15)
-				)
-				(justify mirror)
-			)
-		)
 		(property ki_fp_filters "D*SMA*")
 		(sheetname "/Project Architecture/USB Interface and Power/")
 		(sheetfile "usb_interface.kicad_sch")
-		(attr smd)
+		(attr smd exclude_from_bom dnp)
 		(fp_line
 			(start -3.51 1.65)

Commit message: add eval board
Parts:
- removed JP1: SolderJumper_3_Open, Jumper:SolderJumper-3_P1.3mm_Open_RoundedPad1.0x1.5mm
- added D11: SS13, Diode_SMD:D_SMA, B.Cu at (224.3, 148.4)
- added TP1: ~, DS_Test:TestPoint_0.6mm, F.Cu at (209.2, 134.2)
- added TP10: ~, DS_Test:TestPoint_0.6mm, F.Cu at (220.2, 151.2)
- added TP11: ~, DS_Test:TestPoint_0.6mm, F.Cu at (216.2, 151.2)
- added TP12: ~, DS_Test:TestPoint_0.6mm, B.Cu at (216.4, 128.6)
- added TP13: ~, DS_Test:TestPoint_0.6mm, B.Cu at (214.0, 130.3)
- added TP14: ~, DS_Test:TestPoint_0.6mm, B.Cu at (212.2, 129.2)
- added TP15: ~, DS_Test:TestPoint_0.6mm, F.Cu at (215.3, 129.1)
- added TP16: ~, DS_Test:TestPoint_0.6mm, F.Cu at (224.2, 93.2)
- added TP17: ~, DS_Test:TestPoint_0.6mm, F.Cu at (228.1, 113.2)
- added TP2: ~, DS_Test:TestPoint_0.6mm, F.Cu at (227.7, 97.5)
- added TP3: ~, DS_Test:TestPoint_0.6mm, F.Cu at (211.2, 150.1)
- added TP4: ~, DS_Test:TestPoint_0.6mm, F.Cu at (220.6, 153.2)
- added TP5: ~, DS_Test:TestPoint_0.6mm, F.Cu at (229.2, 122.0)
- added TP6: ~, DS_Test:TestPoint_0.6mm, F.Cu at (214.1, 91.5)
- added TP7: ~, DS_Test:TestPoint_0.6mm, F.Cu at (216.2, 99.8)
- added TP8: ~, DS_Test:TestPoint_0.6mm, F.Cu at (212.7, 152.9)
Connections:
- C36 pad 1: +5V -> VIN_PWR
- C52 pad 1: +5V -> VIN_PWR
- C53 pad 1: +5V -> VIN_PWR
- C83 pad 1: +3.3V -> VIN_PWR
- D2 pad 2: +5V -> VIN_PWR
- D4 pad 1: +5V -> VIN_PWR
- D8 pad 1: +5V -> VIN_PWR
- IC29 pad 3: +3.3V -> VIN_PWR
- IC7 pad 1: +5V -> VIN_PWR
- IC7 pad 2: +5V -> VIN_PWR
- IC7 pad 4: +5V -> VIN_PWR
- IC7 pad 5: +5V -> VIN_PWR
- J1 pad 10: /Project Architecture/PWR -> +3.3V
- J1 pad 12: /Project Architecture/PWR -> +3.3V
- J1 pad 14: /Project Architecture/PWR -> +5V
- J1 pad 16: /Project Architecture/PWR -> +5V
Routing:
- net VIN_PWR: track 0.00 -> 126.7 mm, vias 0 -> 18
- net /Project Architecture/PWR: track 114.1 -> 0.00 mm, vias 6 -> 0
- net +5V: track 87.9 -> 20.3 mm, vias 13 -> 1
- net +3.3V: track 45.9 -> 49.5 mm
- net /Project Architecture/Microcontroller/ADC_VUSB: track 41.2 -> 44.3 mm, vias 2 -> 3
- net VBUS_ISO: track 2.95 -> 5.15 mm
- net +1V1: track 29.3 -> 31.2 mm
- net /Project Architecture/CAN Interface/CAN_TERM_N: track 4.44 -> 6.21 mm
- net /Project Architecture/Microcontroller Peripherals/VREF_IN: track 42.8 -> 44.5 mm
- net /Project Architecture/CAN Interface/CAN_TERM_P: track 4.39 -> 5.95 mm
- net /Project Architecture/USB Interface and Power/FB: track 2.88 -> 4.23 mm
- net GND: track 399.5 -> 400.5 mm, vias 180 -> 177
- net VREF_OUT: track 22.1 -> 23.1 mm
- net /Project Architecture/Microcontroller/CAN_INT: vias 0 -> 1
- added copper zone on B.Cu, net VIN_PWR
- added copper zone on F.Cu, net VIN_PWR
- added copper zone on In3.Cu, net VIN_PWR
- removed copper zone on B.Cu, net +5V
- removed copper zone on F.Cu, net +5V
- removed copper zone on In3.Cu, net +5V
Other:
- board text added: "1V1"
- board text added: "ADCREF"
- board text added: "AUSB"
- board text added: "CANH"
- board text added: "CANL"
- board text added: "CINT"
- board text added: "CRST"
- board text added: "FB"
- board text added: "REF"
- board text added: "VBUSISO"
- board text added: "VIN5V"
- board text added: "VREFO"
- board text removed: "5V"
