File: src/HardwareDesign/1.0.0/can_interface.kicad_sch (KiCad schematic)
At the start: 21 parts, among them IC29 TCAN1044AVDRBRQ1, IC6 MCP2515T-I/ML, X2 16MHz 8pF

Commit message: Update M54C
Parts:
- added R39, R40: 1R 1%, Resistor_SMD:R_0402_1005Metric, symbol DS_Resistor_0402:1R 1% 0402
Connections:
- net CAN_TERM_N: now also R40.1
- net CAN_TERM_P: now also R39.2
- net IC_CAN_N: now also R40.2
- net IC_CAN_P: now also R39.1
Other:
- note added: "Populate R39 and R40 and remove L3, if the CMC degrades signal integrity"

Commit message: add eval board
Parts:
- added TP10, TP11, TP12, TP13: ~, DS_Test:TestPoint_0.6mm, symbol DS_Test:Test_Point
Connections:
- net +3.3V: no longer C83.1, IC29.3 (VCC)
- net CAN_INT: now also TP13.1
- net CAN_RST: now also TP12.1
- net CAN_TERM_N: now also TP11.1
- net CAN_TERM_P: now also TP10.1
- new net VIN_PWR: C83.1, IC29.3 (VCC)
Other:
- moved on the sheet: C33

Commit message: update documentation
Parts:
- TP10, TP11, TP12, TP13: value ~ -> (none)
