File: src/HardwareDesign/1.0.0/microcontroller.kicad_sch (KiCad schematic)
At the start: 32 parts, among them IC1 RP2354B

Commit message: add simple software
Connections:
- net USB_IND renamed HB_IND
Changed lines of the file:
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@@
 		)
 	)
-	(label "USB_IND"
+	(label "HB_IND"
 		(at 121.92 254 0)
 		(effects
