File: src/HardwareDesign/1.0.0/microcontroller_peripherals.kicad_sch (KiCad schematic)
At the start: 45 parts, among them IC1 RP2354B, IC2 AT24C256C-XHL-T, IC3 W25Q128JVPIQ, IC4 MCP6001RT, IC5 LM4040B30FTA, J2 SM03B-SRSS-TB, SW1 B3U-1000P, SW2 B3U-1000P, X1 12MHz 10pF

Commit message: update component list
Parts:
- X1: LCSC_PART C20625731 -> C2901649; MFR YXC Crystal Oscillators -> Shenzhen SCTF Elec; MPN ABM8-272-T3 -> SX3B12.000F1010F30
Changed lines of the file:
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@@
 			)
 		)
-		(property "MFR" "YXC Crystal Oscillators"
+		(property "MFR" "Shenzhen SCTF Elec"
 			(at 296.418 127.762 0)
 			(show_name yes)
@@
 			)
 		)
-		(property "MPN" "ABM8-272-T3"
+		(property "MPN" "SX3B12.000F1010F30"
 			(at 296.418 131.826 0)
 			(show_name yes)
@@
 			)
 		)
-		(property "LCSC_PART" "C20625731"
+		(property "LCSC_PART" "C2901649"
 			(at 296.418 134.112 0)
 			(show_name yes)

Commit message: add eval board
Parts:
- added TP14, TP15, TP16, TP17: ~, DS_Test:TestPoint_0.6mm, symbol DS_Test:Test_Point
Connections:
- net +1V1: now also TP17.1
- net ADC_VREF: now also TP14.1
- net VREF_IN: now also TP16.1
- net VREF_OUT: now also TP15.1

Commit message: update documentation
Parts:
- TP14, TP15, TP16, TP17: value ~ -> (none)
