File: src/HardwareDesign/1.0.0/microcontroller_peripherals.kicad_sch (KiCad schematic)
At the start: 49 parts, among them IC1 RP2354B, IC2 AT24C256C-XHL-T, IC3 W25Q128JVPIQ, IC4 MCP6001RT, IC5 LM4040B30FTA, J2 SM03B-SRSS-TB, SW1 B3U-1000P, SW2 B3U-1000P, X1 12MHz 10pF

Commit message: update generator
Connections:
- net SWCLK: now also J2.1 (SWCLK); no longer J2.3 (SWDAT)
- net SWDIO: now also J2.3 (SWDAT); no longer J2.1 (SWCLK)
Changed lines of the file:
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@@
-	(wire
-		(pts
-			(xy 316.23 85.09) (xy 316.23 69.85)
-		)
-		(stroke
-			(width 0)
-			(type default)
-		)
-	)
 	(wire
 		(pts
@@
 	(wire
 		(pts
-			(xy 318.77 67.31) (xy 339.09 67.31)
+			(xy 316.23 67.31) (xy 339.09 67.31)
 		)
 		(stroke
@@
 	(wire
 		(pts
-			(xy 226.06 85.09) (xy 316.23 85.09)
+			(xy 226.06 85.09) (xy 318.77 85.09)
 		)
 		(stroke
@@
 		(pts
 			(xy 344.17 218.44) (xy 347.98 218.44)
-		)
-		(stroke
-			(width 0)
-			(type default)
-		)
-	)
-	(wire
-		(pts
-			(xy 318.77 87.63) (xy 318.77 67.31)
 		)
 		(stroke
@@
 		)
 	)
+	(label "SWCLK"
+		(at 316.23 69.85 0)
+		(effects
+			(font
+				(size 1.27 1.27)
+			)
+			(justify left bottom)
+		)
+	)
 	(label "XIN"
 		(at 229.87 95.25 0)
@@
 	)
 	(label "SWDIO"
-		(at 229.87 85.09 0)
-		(effects
-			(font
-				(size 1.27 1.27)
-			)
-			(justify left bottom)
+		(at 318.77 85.09 180)
+		(effects
+			(font
+				(size 1.27 1.27)
+			)
+			(justify right bottom)
 		)
 	)
@@
 		)
 	)
+	(label "SWDIO"
+		(at 316.23 67.31 0)
+		(effects
+			(font
+				(size 1.27 1.27)
+			)
+			(justify left bottom)
+		)
+	)
 	(label "QSPI_SS"
 		(at 228.6 114.3 0)
@@
 	)
 	(label "SWCLK"
-		(at 229.87 87.63 0)
-		(effects
-			(font
-				(size 1.27 1.27)
-			)
-			(justify left bottom)
-		)
-	)
+		(at 318.77 87.63 180)
+		(effects
+			(font
+				(size 1.27 1.27)
+			)
+			(justify right bottom)
+		)
+	)
