File: src/HardwareDesign/1.0.0/usb_interface.kicad_sch (KiCad schematic)
At the start: 31 parts, among them IC7 TPS74801DRCT, IC8 SN74LVC1G97QDCKRQ1, IC9 FSUSB42MUX, J3 USB-TYPE-C-018

Commit message: Finalize design
Parts:
- removed C54: 1uF 50V, Capacitor_SMD:C_0402_1005Metric, symbol DS_Capacitor_0402:1uF 50V 0402
- added C36: 4.7uF 25V, Capacitor_SMD:C_0402_1005Metric, symbol DS_Capacitor_0402:4.7uF 25V 0402
- added D10: Green, LED_SMD:LED_0402_1005Metric, symbol DS_Opto:Green_0402
- added R41: 1K 1%, Resistor_SMD:R_0402_1005Metric, symbol DS_Resistor_0402:1K 1% 0402
Connections:
- net BIAS is gone; now on net +5V: IC7.4 (BIAS)
- net +5V: now also D2.2, C36.1
- net GND: now also C36.2, R41.1
- net USB_IND: now also D10.1, R41.2; no longer D2.1, R62.2
- net VBUS: no longer D2.2
- net VBUS_ONBOARD: now also D10.2
- new net 5V_IND: D2.1, R62.2
Other:
- note added: "+5V INDICATOR LED"
- note added: "ONBOARD USB INDICATOR LED"
- note removed: "USB INDICATOR LED"
- moved on the sheet: D2, R62

Commit message: add eval board
Parts:
- added D11: SS13, Diode_SMD:D_SMA, symbol Diode:SS13
- added TP1, TP2, TP3, TP4, TP5, TP6, TP7, TP8: ~, DS_Test:TestPoint_0.6mm, symbol DS_Test:Test_Point
- D8: now fitted; now in the parts list
Connections:
- net +3.3V: now also TP5.1
- net +5V: now also D11.2 (A), TP4.1; no longer C36.1, C52.1, C53.1, D2.2, D4.1 (K), D8.1 (K), IC7.1 (IN), IC7.2 (IN), IC7.4 (BIAS), IC7.5 (EN)
- net ADC_VUSB: now also TP8.1
- net FB: now also TP6.1
- net PGOOD_3V3: now also TP7.1
- net VBUS_ISO: now also TP3.1
- net VBUS_ONBOARD: now also TP2.1
- new net VIN_PWR: C36.1, C52.1, C53.1, D11.1 (K), D2.2, D4.1 (K), D8.1 (K), IC7.1 (IN), IC7.2 (IN), IC7.4 (BIAS), IC7.5 (EN), TP1.1
Other:
- note added: "VBUS_ONBOARD: +5V from the onboard USB-C VBUS_ISO: USB +5V from the M.2 connector +5V: Supply voltage from external source from M.2 connector"
- note removed: "If PGOOD AND PGOOD_3V3 are both 1, Y = 1"

Commit message: update documentation
Parts:
- TP1, TP2, TP3, TP4, TP5, TP6, TP7, TP8: value ~ -> (none)
