File: src/HardwareDesign/M54-DevBoard_1.0.0/USB_and_Power.kicad_sch (KiCad schematic)
At the start: 42 parts, among them IC12 MCP1754ST-3302E/MB, J10 1888687, J8 USB-B-S-F-B-TH, J9 PJ-102AH, T1 SQJ459EP-T1_GE3

Commit message: Generate pdf
Parts:
- IC12: value MCP1754ST-3302E/MB -> MP4462DN-LF-Z; footprint DS_Vreg:SOIC-8_5.3x5.3mm_P1.27mm -> DS_Vreg:SO-8_3.9x4.9mm_EP2.6x3.5mm
- TP1, TP2, TP3, TP4, TP5, TP6, TP7, TP8, TP9: value ~ -> (none)
Connections:
- net GND renamed EP
- net EP: now also IC12.9 (EP)
Other:
- note added: "or B340A-13-F"
- moved on the sheet: C24, C25, C28
