File: src/HardwareDesign/M54-DevBoard_1.0.0/M54-DevBoard_1.0.0.kicad_pcb (KiCad board)
At the start: 4 copper layers, 66 x 147 mm, 119 parts, among them IC1 TXS0108EPWR, IC10 OPA365AQDBVRQ1, IC11 OPA365AQDBVRQ1, IC12 MCP1754ST-3302E/MB, IC13 OPA365AQDBVRQ1, IC2 TXS0108EPWR, IC3 TXS0108EPWR, IC4 TXS0108EPWR, IC5 OPA365AQDBVRQ1, IC6 LM397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

Commit message: Generate pdf
Parts:
- IC12: value MCP1754ST-3302E/MB -> MP4462DN-LF-Z; footprint DS_Vreg:SOIC-8_5.3x5.3mm_P1.27mm -> DS_Vreg:SO-8_3.9x4.9mm_EP2.6x3.5mm
Routing:
- net /Project Architecture/USB and Power/VIN_14V_PROT: track 19.2 -> 21.8 mm
- net /Project Architecture/USB and Power/BUCK_FREQ: track 2.26 -> 3.22 mm
- net /Project Architecture/USB and Power/BUCK_COMP: track 3.22 -> 4.18 mm
- net /Project Architecture/USB and Power/BUCK_EN: track 6.49 -> 7.45 mm
- net GND: track 364.7 -> 365.6 mm, vias 406 -> 412
- net Net-(IC12-FB): track 9.18 -> 9.95 mm
- net Net-(IC12-BST): track 2.03 -> 2.72 mm
- net +5V: vias 76 -> 68

Commit message: fix hardware bugs, add software example
Parts:
- J12: footprint Connector_Dsub:DSUB-9_Socket_Horizontal_P2.77x2.84mm_EdgePinOffset4.94mm_Housed_MountingHolesOffset4.94mm -> Connector_Dsub:DSUB-9_Socket_Horizontal_P2.77x2.84mm_EdgePinOffset7.70mm_Housed_MountingHolesOffset9.12mm
- moved J12 3.47 mm to (234.2, 189.0)
Routing:
- net SHIELD: track 65.9 -> 75.8 mm, vias 0 -> 4
- net GND: track 365.6 -> 360.1 mm, vias 412 -> 403
- net CAN_N: track 98.7 -> 93.4 mm
- net +3.3V: track 258.1 -> 262.4 mm, vias 16 -> 18
- net CAN_P: track 98.8 -> 95.3 mm

Commit message: correct devboard findings
Parts:
- removed IC6: LM397, Package_TO_SOT_SMD:SOT-23-5
- removed the REF** at (215.6, 109.9)
- removed the REF** at (231.2, 118.1)
- removed the REF** at (215.1, 117.9)
- removed the REF** at (224.1, 117.9)
- removed the REF** at (231.4, 110.0)
- added C29: 100nF 50V, DS_Capacitor:C_0603_1608Metric, F.Cu at (219.9, 86.5)
- added IC20: LM397, Package_TO_SOT_SMD:SOT-23-5, F.Cu at (213.8, 89.7)
- added IC21: LM397, Package_TO_SOT_SMD:SOT-23-5, F.Cu at (220.1, 89.7)
- added R24: 10K 1%, DS_Resistor:R_0603_1608Metric, F.Cu at (217.4, 89.7)
- added R25: 10K 1%, DS_Resistor:R_0603_1608Metric, F.Cu at (219.7, 92.8)
- added R26: 10K 1%, DS_Resistor:R_0603_1608Metric, F.Cu at (213.6, 85.1)
- added R27: 10K 1%, DS_Resistor:R_0603_1608Metric, F.Cu at (220.0, 85.0)
- added T2: BSS138LT1G, DS_FET:SOT-23, F.Cu at (227.7, 84.0)
- added T3: BSS138LT1G, DS_FET:SOT-23, F.Cu at (227.7, 88.5)
- added T4: BSS138LT1G, DS_FET:SOT-23, F.Cu at (194.8, 115.2)
- added T5: BSS138LT1G, DS_FET:SOT-23, F.Cu at (194.8, 110.7)
- added T6: BSS138LT1G, DS_FET:SOT-23, F.Cu at (237.6, 115.5)
- added T7: BSS138LT1G, DS_FET:SOT-23, F.Cu at (237.6, 110.6)
- added T8: BSS138LT1G, DS_FET:SOT-23, F.Cu at (196.4, 85.0)
- added T9: BSS138LT1G, DS_FET:SOT-23, F.Cu at (200.9, 85.0)
- R5: value 10K 1% -> 15K 1%; footprint DS_Resistor:R_0402_1005Metric -> DS_Resistor:R_0603_1608Metric
- R6: value 24K 1% -> 10K 1%; footprint DS_Resistor:R_0402_1005Metric -> DS_Resistor:R_0603_1608Metric
- moved R6 23.6 mm to (213.3, 92.5), turned to 0 degrees
- moved R5 18.9 mm to (211.3, 89.7), turned to -90 degrees
- moved C10 15.9 mm to (213.6, 86.6), turned to 0 degrees
- moved J10 0.56 mm to (235.7, 59.0)
Connections:
- D10 pad 1: GND -> Net-(D10-Pad1)
- D2 pad 1: GND -> Net-(D2-Pad1)
- D3 pad 1: VCOMP -> Net-(D3-Pad1)
- D4 pad 1: VCOMP -> Net-(D4-Pad1)
- D5 pad 1: GND -> Net-(D5-Pad1)
- D6 pad 1: VCOMP -> Net-(D6-Pad1)
- D8 pad 1: GND -> Net-(D8-Pad1)
- D9 pad 1: VCOMP -> Net-(D9-Pad1)
- J1 pad SH1: (no net) -> GND
- R11 pad 1: VCOMP -> +5V
- R4 pad 1: VCOMP -> +5V
- R7 pad 1: VCOMP -> +5V
- R9 pad 1: VCOMP -> +5V
Routing:
- net VDD: track 52.0 -> 235.1 mm, vias 7 -> 8
- net VCOMP: track 152.2 -> 0.00 mm, vias 2 -> 0
- net 3.3V_LED: track 0.00 -> 107.0 mm, vias 0 -> 2
- net 5V_LED: track 0.00 -> 98.8 mm, vias 0 -> 6
- net +5V: track 288.3 -> 349.5 mm, vias 68 -> 69
- net Net-(D9-Pad1): track 0.00 -> 24.5 mm
- net Net-(D10-Pad1): track 0.00 -> 20.9 mm
- net GND: track 360.1 -> 378.1 mm, vias 403 -> 401
- net Net-(D3-Pad1): track 0.00 -> 17.6 mm
- net VREF: track 3.62 -> 20.5 mm
- net Net-(D2-Pad1): track 0.00 -> 13.1 mm
- net Net-(D8-Pad1): track 0.00 -> 10.0 mm
- net Net-(D6-Pad1): track 0.00 -> 10.0 mm
- net Net-(D5-Pad1): track 0.00 -> 9.59 mm
- net Net-(D4-Pad1): track 0.00 -> 9.56 mm
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