File: src/HardwareDesign/M54-DevBoard_1.0.0/Output_interfaces.kicad_sch (KiCad schematic)
At the start: 54 parts, among them IC1 TXS0108EPWR, IC10 OPA365AQDBVRQ1, IC11 OPA365AQDBVRQ1, IC13 OPA365AQDBVRQ1, IC2 TXS0108EPWR, IC3 TXS0108EPWR, IC4 TXS0108EPWR, IC5 OPA365AQDBVRQ1, IC6 LM397, IC7 OPA365AQDBVRQ1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

Commit message: Generate pdf
Parts:
- D16, TP10, TP11, TP12: value ~ -> (none)

Commit message: scope measurements
Parts:
- renumbered IC6 to U6

Commit message: correct devboard findings
Parts:
- removed R5: 10K 1%, DS_Resistor:R_0402_1005Metric, symbol DS_Resistor_0402:10K 1% 0402
- removed R6: 24K 1%, DS_Resistor:R_0402_1005Metric, symbol DS_Resistor_0402:24K 1% 0402
- added C29: 100nF 50V, DS_Capacitor:C_0603_1608Metric, symbol DS_Capacitor_0603:100nF 50V 0603
- added IC21: LM397, Package_TO_SOT_SMD:SOT-23-5, symbol Comparator:LM397
- added R24, R25, R26, R27, R6: 10K 1%, DS_Resistor:R_0603_1608Metric, symbol DS_Resistor_0603:10K 1% 0603
- added R5: 15K 1%, DS_Resistor:R_0603_1608Metric, symbol DS_Resistor_0603:15K 1% 0603
- added T2, T3, T4, T5, T6, T7, T8, T9: BSS138LT1G, DS_FET:SOT-23, symbol DS_FET:BSS138LT1G
- renumbered U6 to IC20
Connections:
- net +5V: now also R11.1, R4.1, R7.1, R9.1, C29.1, IC21.5 (V+), R26.1, R27.1, R5.1
- net GND: now also C29.2, IC21.2 (V-), R25.2, R6.2, T2.2, T3.2, T4.2, T5.2, T6.2, T7.2, T8.2, T9.2; no longer D10.1, D2.1, D5.1, D8.1
- net VDD: now also R24.1; no longer IC20.3 (+)
- net VREF: now also IC21.3 (+), R5.2, R6.1
- removed net VCOMP: D3.1, D4.1, D6.1, D9.1, IC20.4, R11.1, R4.1, R7.1, R9.1
- new net: D3.1, T9.3
- new net: D4.1, T7.3
- new net: D5.1, T6.3
- new net: D6.1, T5.3
- new net: D2.1, T8.3
- new net: D8.1, T4.3
- new net: D9.1, T2.3
- new net: D10.1, T3.3
- new net 3.3V_LED: IC21.4, R27.2, T3.1, T4.1, T6.1, T8.1
- new net 5V_LED: IC20.4, R26.2, T2.1, T5.1, T7.1, T9.1
- new net VDD_SENSE: IC20.3 (+), IC21.1 (-), R24.2, R25.1
Other:
- note added: "1.65V"
- note added: "2.0V"
- note added: "2.5V"
- note added: "Simple comparator. VREF = 2.0V If VDD > VREF -> HiZ If VDD < VREF -> LOW"
- note added: "V+ > V- (2.0V > 1.65V) -> HiZ -> Tgate = High -> 3.3V LED ON V+ < V- (2.0V < 2.5V) -> LOW -> Tgate = LOW -> 3.3V LED OFF"
- note added: "V+ > V- (2.5V > 2.0V) -> HiZ -> Tgate = High -> 5V LED ON V+ < V- (1.65V < 2.0V) -> LOW -> Tgate = LOW -> 5V LED OFF"
- note removed: "Simple comparator. VREF = 3.53V If VDD > VREF -> HIGH If VDD < VREF -> LOW If 5V -> VCOMP = HIGH If 3.3V -> VCOMP = LOW"
- moved on the sheet: C10, D2, D3, D4, D5, IC1, IC20, IC3, J11, R3, R4, R7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
